File: hardware/RealRollOverDetection.kicad_sch (KiCad schematic)
At the start: 23 parts, among them J1 AVR-UPDI-6, J2 Conn_02x01, U1 ATtiny1617-M, U2 MPU-6050

Commit message: Updated with comments
Parts:
- added C3: 1uF, Capacitor_SMD:C_0603_1608Metric, symbol Device:C
- added C4: 10uF, Capacitor_SMD:C_0603_1608Metric, symbol Device:C
- added C5, C6, C7: 100uF, Capacitor_SMD:C_0603_1608Metric, symbol Device:C
- C1: value 100n -> 1uF
- C2: value 10n -> 10uF
Connections:
- net GND: now also C7.2; no longer J2.1 (Pin_1)
- net at C1.1, C2.1, J2.2 (Pin_2)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: now also C7.1
- net at U2.13 (VDD): now also U2.8 (VLOGIC), C3.2, C4.2, C5.2, C6.2
- new net +3.3V: C3.1, C4.1, C5.1, C6.1, J2.1 (Pin_1)
- no-connect marks 0 -> 18
Other:
- note added: "Things to solve: - connections to MPU6050 - does the debugger provide power (3.3V or sth like that) - when debugger not connected then where does the 3.3V come from possibly just 3.3V and GND line? As no data is needed to be transferred to other boards"
- moved on the sheet: C1, C2, J2, U2
